File: kicad/piaxe.kicad_pcb (KiCad board)
At the start: 4 copper layers, 89 x 134 mm, 200 parts, among them J1 Barrel_Jack_Switch, J2 Conn_01x06, J3 SWD, M2 Fan_4pin, P1 MYUSB_B, Q1 BSS138, Q3 CSD16415Q5T, Q4 CSD16415Q5T, Q5 CSD16415Q5T, Q6 CSD16415Q5T, Q7 BSS138, U19 BM1366_mode1, U20 BM1366_mode1, U25 BM1366_mode1, U26 BM1366_mode1, U29 2N7001TDCK, U3 LTC3856, U30 2N7001TDCK, U32 STM32L052K6Tx, U33 TMP1075, U4 MCP1824T-0802E, U6 AP3211, U7 MCP1824T-1802E, U8 25MHz

Commit message: added 3d models
Parts:
- added REF**: heatsink, myfootprints:dummy, F.Cu at (81.7, 70.4)
Changed lines of the file:
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@@
     (pad "30" smd rect locked (at 0 1.108 270) (size 4.277 4.53) (layers "F.Cu" "F.Mask")
       (net 1 "GND") (pinfunction "GND") (pintype "input") (thermal_bridge_angle 45))
-    (model "${KIPRJMOD}/../3d/heatsink-40x40.step" hide
-      (offset (xyz -19.75 -19.25 0.8))
+    (model "/home/thomas/git/quadaxe/3d/bm1366.step"
+      (offset (xyz 0 0 0.3))
       (scale (xyz 1 1 1))
-      (rotate (xyz 0 0 0))
+      (rotate (xyz 0 0 -90))
     )
   )
@@
     (pad "2" smd rect (at 3.805 0) (size 3.3 2.8) (layers "F.Cu" "F.Paste" "F.Mask")
       (net 64 "Net-(L1-Pad2)") (pinfunction "2") (pintype "passive") (thermal_bridge_angle 45))
+    (model "/home/thomas/git/quadaxe/3d/FP1006V2-R.STEP"
+      (offset (xyz 3 -7.5 10))
+      (scale (xyz 1 1 1))
+      (rotate (xyz 0 180 0))
+    )
   )
   (footprint "Resistor_SMD:R_0805_2012Metric" (layer "F.Cu")
@@
         (effects (font (size 0.8 0.8) (thickness 0.15)))
     )
-    (fp_text value "MountingHole_3.2mm_M3_Pad_Via" (at 0 4.2) (layer "F.Fab")
+    (fp_text value "MountingHole_3.2mm_M3_Pad_Via" (at 0 4.2) (layer "F.Fab") hide
         (effects (font (size 1 1) (thickness 0.15)))
     )
@@
         (effects (font (size 0.8 0.8) (thickness 0.15)))
     )
-    (fp_text value "MountingHole_3.2mm_M3" (at 0 4.2) (layer "F.Fab")
+    (fp_text value "MountingHole_3.2mm_M3" (at 0 4.2) (layer "F.Fab") hide
         (effects (font (size 1 1) (thickness 0.15)))
     )
@@
       (rotate (xyz 0 0 0))
     )
+    (model "/home/thomas/git/quadaxe/3d/AB2_SON5x6MM.wrl"
+      (offset (xyz 0 0 0))
+      (scale (xyz 0.39 0.39 1))
+      (rotate (xyz 0 0 0))
+    )
   )
   (footprint "LED_SMD:LED_1206_3216Metric" (layer "F.Cu")
@@
     (pad "6" smd rect (at 2.975 -0.565 180) (size 1.825 0.7) (layers "F.Cu" "F.Paste" "F.Mask")
       (net 1 "GND") (pinfunction "shield") (pintype "passive"))
-    (model "${KICAD6_3DMODEL_DIR}/Connector_USB.3dshapes/USB_Micro-B_Amphenol_10103594-0001LF_Horizontal.wrl"
-      (offset (xyz 0 0 0))
+    (model "/home/thomas/git/quadaxe/3d/10103594.step"
+      (offset (xyz 0 0 1.5))
       (scale (xyz 1 1 1))
-      (rotate (xyz 0 0 0))
+      (rotate (xyz 90 0 180))
     )
   )
@@
         (effects (font (size 0.8 0.8) (thickness 0.15)))
     )
-    (fp_text value "MountingHole_3.2mm_M3" (at 0 4.2) (layer "F.Fab")
+    (fp_text value "MountingHole_3.2mm_M3" (at 0 4.2) (layer "F.Fab") hide
         (effects (font (size 1 1) (thickness 0.15)))
     )
@@
         (effects (font (size 0.8 0.8) (thickness 0.15)))
     )
-    (fp_text value "MountingHole_3.2mm_M3" (at 0 4.2) (layer "F.Fab")
+    (fp_text value "MountingHole_3.2mm_M3" (at 0 4.2) (layer "F.Fab") hide
         (effects (font (size 1 1) (thickness 0.15)))
     )
@@
       (rotate (xyz 0 0 0))
     )
+    (model "/home/thomas/git/quadaxe/3d/AB2_SON5x6MM.wrl"
+      (offset (xyz 0 0 0))
+      (scale (xyz 0.39 0.39 1))
+      (rotate (xyz 0 0 0))
+    )
   )
   (footprint "Capacitor_SMD:C_0805_2012Metric" (layer "F.Cu")
@@
         (effects (font (size 0.8 0.8) (thickness 0.15)))
     )
-    (fp_text value "MountingHole_3.2mm_M3_Pad_Via" (at 0 4.2) (layer "F.Fab")
+    (fp_text value "MountingHole_3.2mm_M3_Pad_Via" (at 0 4.2) (layer "F.Fab") hide
         (effects (font (size 1 1) (thickness 0.15)))
     )
@@
       (rotate (xyz 0 0 0))
     )
+    (model "/home/thomas/git/quadaxe/3d/AB2_SON5x6MM.wrl"
+      (offset (xyz 0 0 0))
+      (scale (xyz 0.39 0.39 1))
+      (rotate (xyz 0 0 0))
+    )
   )
   (footprint "Resistor_SMD:R_0805_2012Metric" (layer "F.Cu")
@@
         (effects (font (size 0.8 0.8) (thickness 0.15)))
     )
-    (fp_text value "MountingHole_3.2mm_M3" (at 0 4.2) (layer "F.Fab")
+    (fp_text value "MountingHole_3.2mm_M3" (at 0 4.2) (layer "F.Fab") hide
         (effects (font (size 1 1) (thickness 0.15)))
     )
@@
     (pad "30" smd rect (at 0 1.108 270) (size 4.277 4.53) (layers "F.Cu" "F.Mask")
       (net 1 "GND") (pinfunction "GND") (pintype "input") (thermal_bridge_angle 45))
+    (model "/home/thomas/git/quadaxe/3d/bm1366.step"
+      (offset (xyz 0 0 0.3))
+      (scale (xyz 1 1 1))
+      (rotate (xyz 0 0 -90))
+    )
   )
   (footprint "Capacitor_SMD:C_0805_2012Metric" (layer "F.Cu")
@@
         (effects (font (size 0.8 0.8) (thickness 0.15)))
     )
-    (fp_text value "MountingHole_3.2mm_M3_Pad_Via" (at 0 4.2) (layer "F.Fab")
+    (fp_text value "MountingHole_3.2mm_M3_Pad_Via" (at 0 4.2) (layer "F.Fab") hide
         (effects (font (size 1 1) (thickness 0.15)))
     )
@@
     (pad "30" smd rect (at 0 1.108 90) (size 4.277 4.53) (layers "F.Cu" "F.Mask")
       (net 1 "GND") (pinfunction "GND") (pintype "input") (thermal_bridge_angle 45))
+    (model "/home/thomas/git/quadaxe/3d/bm1366.step"
+      (offset (xyz 0 0 0.3))
+      (scale (xyz 1 1 1))
+      (rotate (xyz 0 0 -90))
+    )
   )
   (footprint "Capacitor_SMD:C_0805_2012Metric" (layer "F.Cu")
@@
         (effects (font (size 0.8 0.8) (thickness 0.15)))
     )
-    (fp_text value "MountingHole_3.2mm_M3_Pad_Via" (at 0 4.2) (layer "F.Fab")
+    (fp_text value "MountingHole_3.2mm_M3_Pad_Via" (at 0 4.2) (layer "F.Fab") hide
         (effects (font (size 1 1) (thickness 0.15)))
     )
@@
     (pad "30" smd rect (at 0 1.108 90) (size 4.277 4.53) (layers "F.Cu" "F.Mask")
       (net 1 "GND") (pinfunction "GND") (pintype "input") (thermal_bridge_angle 45))
+    (model "/home/thomas/git/quadaxe/3d/bm1366.step"
+      (offset (xyz 0 0 0.3))
+      (scale (xyz 1 1 1))
+      (rotate (xyz 0 0 -90))
+    )
   )
   (footprint "MountingHole:MountingHole_3.2mm_M3_Pad_Via" locked (layer "F.Cu")
@@
         (effects (font (size 0.8 0.8) (thickness 0.15)))
     )
-    (fp_text value "MountingHole_3.2mm_M3_Pad_Via" (at 0 4.2) (layer "F.Fab")
+    (fp_text value "MountingHole_3.2mm_M3_Pad_Via" (at 0 4.2) (layer "F.Fab") hide
         (effects (font (size 1 1) (thickness 0.15)))
     )
@@
       (net 23 "Net-(C23-Pad1)") (pinfunction "1") (pintype "passive"))
   )
+  (footprint "myfootprints:dummy" (layer "F.Cu")
+    (at 81.7 70.4)
+    (attr through_hole)
+    (fp_text reference "REF**" (at 0 1.5) (layer "F.SilkS") hide
+        (effects (font (size 1 1) (thickness 0.15)))
+    )
+    (fp_text value "heatsink" (at 0 -1.5) (layer "F.Fab") hide
+        (effects (font (size 1 1) (thickness 0.15)))
+    )
+    (fp_circle (center 0 0) (end 0.5 0)
+      (stroke (width 0.12) (type solid)) (fill none) (layer "Eco1.User"))
+    (pad "" smd circle (at 0 0) (size 1.524 1.524) (layers "Dwgs.User"))
+    (model "/home/thomas/git/quadaxe/3d/heatsink-13x12x5.step"
+      (offset (xyz 0 0 5))
+      (scale (xyz 1 1 1))
+      (rotate (xyz 0 0 0))
+    )
+  )
   (footprint "Connector_BarrelJack:BarrelJack_CUI_PJ-102AH_Horizontal" (layer "F.Cu")
     (at 65 53.2 180)
@@
     (pad "2" smd rect (at 3.805 0) (size 3.3 2.8) (layers "F.Cu" "F.Paste" "F.Mask")
       (net 56 "Net-(L2-Pad2)") (pinfunction "2") (pintype "passive") (thermal_bridge_angle 45))
+    (model "/home/thomas/git/quadaxe/3d/FP1006V2-R.STEP"
+      (offset (xyz 3 -7.5 10))
+      (scale (xyz 1 1 1))
+      (rotate (xyz 0 180 0))
+    )
   )
   (footprint "Package_DFN_QFN:QFN-32-1EP_5x5mm_P0.5mm_EP3.45x3.45mm_ThermalVias" (layer "F.Cu")
@@
       (rotate (xyz 0 0 0))
     )
+    (model "/home/thomas/git/quadaxe/3d/AB2_SON5x6MM.wrl"
+      (offset (xyz 0 0 0))
+      (scale (xyz 0.39 0.39 1))
+      (rotate (xyz 0 0 0))
+    )
   )
   (footprint "Capacitor_SMD:C_1210_3225Metric" (layer "F.Cu")
@@
         (effects (font (size 0.8 0.8) (thickness 0.15)))
     )
-    (fp_text value "MountingHole_3.2mm_M3_Pad_Via" (at 0 4.2) (layer "F.Fab")
+    (fp_text value "MountingHole_3.2mm_M3_Pad_Via" (at 0 4.2) (layer "F.Fab") hide
         (effects (font (size 1 1) (thickness 0.15)))
     )
