File: kicad/power.kicad_sch (KiCad schematic)
At the start: 72 parts, among them Q3 CSD16415Q5T, Q4 CSD16415Q5T, Q7 CSD16415Q5T, Q8 CSD16415Q5T, U17 LTC3856, U3 AP3211, U4 +0V8, U5 MCP1824T-1802E, U6 MCP1824T-0802E

Commit message: v0.02
Parts:
- added C24: 22µ/16V, Capacitor_SMD:C_1206_3216Metric, symbol Device:C
- added C9: 10µF/50V, Capacitor_SMD:C_1206_3216Metric, symbol Device:C
- added NT7: NetTie_2, myfootprints:NetTie-2_L3_SMD_Pad0.5mm, symbol Device:NetTie_2
- added U36: NCP1117ST33, Package_TO_SOT_SMD:SOT-223-3_TabPin2, symbol Regulator_Linear:AZ1117-3.3
- C55, C56, C58, C59: Manufacturer C1210C476M9PAC7800 -> C1210C107M9PAC7800; OrderNr 399-C1210C476M9PAC7800CT-ND -> 399-C1210C107M9PAC7800CT-ND
- C95: Manufacturer 875075561008 -> 875075355002; OrderNr 732-6502-1-ND -> 732-6489-1-ND
- R24: value 49,9k -> 84.5k
Connections:
- net +3V3: now also C24.1, U36.2 (VO); no longer R26.2
- net GND: now also C24.2, C9.2, NT7.2, U36.1 (GND); no longer C64.2, C65.2, R23.1, R25.1, R25.1, R27.2, R28.2
- new net +5V: C9.1, R26.2, U36.3 (VI)
- new net GNDA: C64.2, C65.2, NT7.1, R23.1, R25.1, R25.1, R27.2, R28.2
Other:
- moved on the sheet: C15, C24, C9, D9, L1, R24, R25, R26, TP2, U3

Commit message: push
Parts:
- U36: Distributor D -> (none)
Changed lines of the file:
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@@
       (effects (font (size 1.27 1.27)) hide)
     )
-    (property "Distributor" "D" (at 378.46 166.37 0)
+    (property "Distributor" "" (at 378.46 166.37 0)
       (effects (font (size 1.27 1.27)) hide)
     )
