File: kicad/piaxe.kicad_sch (KiCad schematic)
At the start: 4 parts, among them J3 Barrel_Jack_Switch

Commit message: v0.02
Connections:
- net Power/VIn renamed Power/+12V
Other:
- sheet Power ports: added +12V, +5V; removed VIn
- sheet STM32 ports: added +12V, +5V; removed none
Changed lines of the file:
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@@
   (junction (at 43.815 57.15) (diameter 0) (color 0 0 0 0)
   )
+  (junction (at 77.47 52.07) (diameter 0) (color 0 0 0 0)
+  )
   (wire (pts (xy 111.76 75.565) (xy 74.295 75.565))
     (stroke (width 0) (type default))
@@
     (stroke (width 0) (type default))
   )
+  (wire (pts (xy 136.525 45.085) (xy 136.525 74.93))
+    (stroke (width 0) (type default))
+  )
+  (wire (pts (xy 77.47 45.085) (xy 136.525 45.085))
+    (stroke (width 0) (type default))
+  )
   (wire (pts (xy 110.49 52.07) (xy 110.49 74.295))
     (stroke (width 0) (type default))
@@
     (stroke (width 0) (type default))
   )
+  (wire (pts (xy 77.47 52.07) (xy 77.47 45.085))
+    (stroke (width 0) (type default))
+  )
   (wire (pts (xy 71.755 93.345) (xy 82.55 93.345))
     (stroke (width 0) (type default))
@@
     (stroke (width 0) (type default))
   )
+  (wire (pts (xy 135.255 76.835) (xy 144.78 76.835))
+    (stroke (width 0) (type default))
+  )
   (wire (pts (xy 144.78 78.74) (xy 133.985 78.74))
     (stroke (width 0) (type default))
@@
     (stroke (width 0) (type default))
   )
+  (wire (pts (xy 99.695 59.69) (xy 135.255 59.69))
+    (stroke (width 0) (type default))
+  )
+  (wire (pts (xy 135.255 59.69) (xy 135.255 76.835))
+    (stroke (width 0) (type default))
+  )
   (wire (pts (xy 133.985 78.74) (xy 133.985 57.785))
     (stroke (width 0) (type default))
@@
     (stroke (width 0) (type default))
   )
+  (wire (pts (xy 77.47 52.07) (xy 82.55 52.07))
+    (stroke (width 0) (type default))
+  )
   (wire (pts (xy 113.03 55.88) (xy 113.03 76.835))
     (stroke (width 0) (type default))
@@
     (stroke (width 0) (type default))
   )
+  (wire (pts (xy 136.525 74.93) (xy 144.78 74.93))
+    (stroke (width 0) (type default))
+  )
   (wire (pts (xy 99.695 55.88) (xy 113.03 55.88))
     (stroke (width 0) (type default))
@@
     (stroke (width 0) (type default))
   )
-  (wire (pts (xy 55.245 52.07) (xy 82.55 52.07))
+  (wire (pts (xy 55.245 52.07) (xy 77.47 52.07))
     (stroke (width 0) (type default))
   )
   (wire (pts (xy 99.695 66.04) (xy 131.445 66.04))
     (stroke (width 0) (type default))
-  )
-  (symbol (lib_id "power:+3V3") (at 55.245 182.88 180) (unit 1)
-    (in_bom yes) (on_board yes) (dnp no) (fields_autoplaced)
-    (property "Reference" "#PWR05" (at 55.245 179.07 0)
-      (effects (font (size 1.27 1.27)) hide)
-    )
-    (property "Value" "+3V3" (at 55.245 187.96 0)
-      (effects (font (size 1.27 1.27)))
-    )
-    (property "Footprint" "" (at 55.245 182.88 0)
-      (effects (font (size 1.27 1.27)) hide)
-    )
-    (property "Datasheet" "" (at 55.245 182.88 0)
-      (effects (font (size 1.27 1.27)) hide)
-    )
-    (pin "1")
-    (instances
-      (project "piaxe"
-        (path "/e63e39d7-6ac0-4ffd-8aa3-1841a4541b55"
-          (reference "#PWR05") (unit 1)
-        )
-      )
-    )
-  )
-  (symbol (lib_id "power:+5V") (at 43.18 182.88 180) (unit 1)
-    (in_bom yes) (on_board yes) (dnp no) (fields_autoplaced)
-    (property "Reference" "#PWR02" (at 43.18 179.07 0)
-      (effects (font (size 1.27 1.27)) hide)
-    )
-    (property "Value" "+5V" (at 43.18 187.96 0)
-      (effects (font (size 1.27 1.27)))
-    )
-    (property "Footprint" "" (at 43.18 182.88 0)
-      (effects (font (size 1.27 1.27)) hide)
-    )
-    (property "Datasheet" "" (at 43.18 182.88 0)
-      (effects (font (size 1.27 1.27)) hide)
-    )
-    (pin "1")
-    (instances
-      (project "piaxe"
-        (path "/e63e39d7-6ac0-4ffd-8aa3-1841a4541b55"
-          (reference "#PWR02") (unit 1)
-        )
-      )
-    )
   )
   (symbol (lib_id "power:GND") (at 55.245 66.675 0) (unit 1)
@@
     )
   )
-  (symbol (lib_id "power:PWR_FLAG") (at 43.18 182.88 0) (unit 1)
-    (in_bom yes) (on_board yes) (dnp no) (fields_autoplaced)
-    (property "Reference" "#FLG02" (at 43.18 180.975 0)
-      (effects (font (size 1.27 1.27)) hide)
-    )
-    (property "Value" "PWR_FLAG" (at 43.18 178.435 0)
-      (effects (font (size 1.27 1.27)))
-    )
-    (property "Footprint" "" (at 43.18 182.88 0)
-      (effects (font (size 1.27 1.27)) hide)
-    )
-    (property "Datasheet" "~" (at 43.18 182.88 0)
-      (effects (font (size 1.27 1.27)) hide)
-    )
-    (pin "1")
-    (instances
-      (project "piaxe"
-        (path "/e63e39d7-6ac0-4ffd-8aa3-1841a4541b55"
-          (reference "#FLG02") (unit 1)
-        )
-      )
-    )
-  )
   (symbol (lib_id "Diode:5KPxxA") (at 55.245 58.42 270) (unit 1)
     (in_bom yes) (on_board yes) (dnp no)
@@
         (path "/e63e39d7-6ac0-4ffd-8aa3-1841a4541b55"
           (reference "#PWR03") (unit 1)
-        )
-      )
-    )
-  )
-  (symbol (lib_id "power:+12V") (at 32.385 182.88 180) (unit 1)
-    (in_bom yes) (on_board yes) (dnp no) (fields_autoplaced)
-    (property "Reference" "#PWR01" (at 32.385 179.07 0)
-      (effects (font (size 1.27 1.27)) hide)
-    )
-    (property "Value" "+12V" (at 32.385 187.96 0)
-      (effects (font (size 1.27 1.27)))
-    )
-    (property "Footprint" "" (at 32.385 182.88 0)
-      (effects (font (size 1.27 1.27)) hide)
-    )
-    (property "Datasheet" "" (at 32.385 182.88 0)
-      (effects (font (size 1.27 1.27)) hide)
-    )
-    (pin "1")
-    (instances
-      (project "piaxe"
-        (path "/e63e39d7-6ac0-4ffd-8aa3-1841a4541b55"
-          (reference "#PWR01") (unit 1)
-        )
-      )
-    )
-  )
-  (symbol (lib_id "power:PWR_FLAG") (at 32.385 182.88 0) (unit 1)
-    (in_bom yes) (on_board yes) (dnp no)
-    (property "Reference" "#FLG01" (at 32.385 180.975 0)
-      (effects (font (size 1.27 1.27)) hide)
-    )
-    (property "Value" "PWR_FLAG" (at 32.385 178.435 0)
-      (effects (font (size 1.27 1.27)))
-    )
-    (property "Footprint" "" (at 32.385 182.88 0)
-      (effects (font (size 1.27 1.27)) hide)
-    )
-    (property "Datasheet" "~" (at 32.385 182.88 0)
-      (effects (font (size 1.27 1.27)) hide)
-    )
-    (pin "1")
-    (instances
-      (project "piaxe"
-        (path "/e63e39d7-6ac0-4ffd-8aa3-1841a4541b55"
-          (reference "#FLG01") (unit 1)
-        )
-      )
-    )
-  )
-  (symbol (lib_id "power:PWR_FLAG") (at 55.245 182.88 0) (unit 1)
-    (in_bom yes) (on_board yes) (dnp no) (fields_autoplaced)
-    (property "Reference" "#FLG03" (at 55.245 180.975 0)
-      (effects (font (size 1.27 1.27)) hide)
-    )
-    (property "Value" "PWR_FLAG" (at 55.245 178.435 0)
-      (effects (font (size 1.27 1.27)))
-    )
-    (property "Footprint" "" (at 55.245 182.88 0)
-      (effects (font (size 1.27 1.27)) hide)
-    )
-    (property "Datasheet" "~" (at 55.245 182.88 0)
-      (effects (font (size 1.27 1.27)) hide)
-    )
-    (pin "1")
-    (instances
-      (project "piaxe"
-        (path "/e63e39d7-6ac0-4ffd-8aa3-1841a4541b55"
-          (reference "#FLG03") (unit 1)
         )
       )
@@
       (effects (font (size 1.27 1.27)) (justify left top))
     )
-    (pin "VIn" input (at 82.55 52.07 180)
-      (effects (font (size 1.27 1.27)) (justify left))
-    )
     (pin "+1V2" output (at 99.695 52.07 0)
       (effects (font (size 1.27 1.27)) (justify right))
@@
     (pin "1V2_RUN" input (at 99.695 64.135 0)
       (effects (font (size 1.27 1.27)) (justify right))
+    )
+    (pin "+5V" output (at 99.695 59.69 0)
+      (effects (font (size 1.27 1.27)) (justify right))
+    )
+    (pin "+12V" input (at 82.55 52.07 180)
+      (effects (font (size 1.27 1.27)) (justify left))
     )
     (instances
@@
       (effects (font (size 1.27 1.27)) (justify left))
     )
+    (pin "+12V" input (at 144.78 74.93 180)
+      (effects (font (size 1.27 1.27)) (justify left))
+    )
+    (pin "+5V" input (at 144.78 76.835 180)
+      (effects (font (size 1.27 1.27)) (justify left))
+    )
