File: kicad/pi.kicad_sch (KiCad schematic)
At the start: 13 parts, among them J1 Conn_02x20_Odd_Even, M1 Fan_4pin, U13 TMP1075

Commit message: switched pinheader on top to pinsocket on bottom
Parts:
- J1: footprint Connector_PinHeader_2.54mm:PinHeader_2x20_P2.54mm_Vertical -> Connector_PinSocket_2.54mm:PinSocket_2x20_P2.54mm_Vertical
Changed lines of the file:
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@@
       (effects (font (size 1.27 1.27)) hide)
     )
-    (property "Footprint" "Connector_PinHeader_2.54mm:PinHeader_2x20_P2.54mm_Vertical" (at 184.15 93.98 0)
+    (property "Footprint" "Connector_PinSocket_2.54mm:PinSocket_2x20_P2.54mm_Vertical" (at 184.15 93.98 0)
       (effects (font (size 1.27 1.27)) hide)
     )
